File: PCB/Power.kicad_sch (KiCad schematic)
At the start: 47 parts, among them Q201 IRFR7440TRPBF, Q202 IRFR7440TRPBF, U201 LM25118, U202 XC6206PxxxMR, U203 WS3222D, U204 WS3222D

Commit message: Final fixes before production
Parts:
- R208, R209: LCSC C105871 -> C25867
- U201: symbol Skrooter_symbols:LM25118 -> Skrooterlib:LM25118
- U203, U204: symbol Skrooter_symbols:WS3222D -> Skrooterlib:WS3222D
Changed lines of the file:
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@@
-    )
-  )
-  (symbol (lib_id "power:PWR_FLAG") (at 46.99 22.86 0) (mirror y) (unit 1)
-    (in_bom yes) (on_board yes) (dnp no) (fields_autoplaced)
-    (property "Reference" "#FLG0201" (at 46.99 20.955 0)
-      (effects (font (size 1.27 1.27)) hide)
-    )
-    (property "Value" "PWR_FLAG" (at 46.99 19.2842 0)
-      (effects (font (size 1.27 1.27)))
-    )
-    (property "Footprint" "" (at 46.99 22.86 0)
-      (effects (font (size 1.27 1.27)) hide)
-    )
-    (property "Datasheet" "~" (at 46.99 22.86 0)
-      (effects (font (size 1.27 1.27)) hide)
-    )
-    (pin "1")
-    (instances
-      (project "SmallLedPlatform"
-        (path "/84eef422-4118-4730-b7a0-1fdaa916c3b4/d71115cb-c282-4713-80a7-e4f7bd9dfc70"
-          (reference "#FLG0201") (unit 1)
-        )
-      )
     )
   )
@@
       (effects (font (size 1.27 1.27)) hide)
     )
-    (property "LCSC" "C105871" (at 261.62 74.93 0)
+    (property "LCSC" "C25867" (at 261.62 74.93 0)
       (effects (font (size 1.27 1.27)) hide)
     )
@@
     )
   )
-  (symbol (lib_id "Skrooter_symbols:WS3222D") (at 128.27 137.16 0) (unit 1)
+  (symbol (lib_id "Skrooterlib:WS3222D") (at 128.27 137.16 0) (unit 1)
     (in_bom yes) (on_board yes) (dnp no) (fields_autoplaced)
     (property "Reference" "U203" (at 128.905 133.511 0)
@@
     )
   )
-  (symbol (lib_id "Skrooter_symbols:WS3222D") (at 128.27 165.1 0) (unit 1)
+  (symbol (lib_id "Skrooterlib:WS3222D") (at 128.27 165.1 0) (unit 1)
     (in_bom yes) (on_board yes) (dnp no) (fields_autoplaced)
     (property "Reference" "U204" (at 128.905 161.451 0)
@@
       (effects (font (size 1.27 1.27)) hide)
     )
-    (property "LCSC" "C105871" (at 232.41 74.93 0)
+    (property "LCSC" "C25867" (at 232.41 74.93 0)
       (effects (font (size 1.27 1.27)) hide)
     )
@@
     )
   )
-  (symbol (lib_id "Skrooter_symbols:LM25118") (at 118.11 21.59 0) (unit 1)
+  (symbol (lib_id "Skrooterlib:LM25118") (at 118.11 21.59 0) (unit 1)
     (in_bom yes) (on_board yes) (dnp no) (fields_autoplaced)
     (property "Reference" "U201" (at 118.11 17.941 0)
@@
       (effects (font (size 1.27 1.27)))
     )
-    (property "Footprint" "Package_SO:HTSSOP-20-1EP_4.4x6.5mm_P0.65mm_EP3.4x6.5mm_Mask2.75x3.43mm_ThermalVias" (at 116.84 30.48 0)
-      (effects (font (size 1.27 1.27)) hide)
-    )
+    (property "Footprint" "Package_SO:HTSSOP-20-1EP_4.4x6.5mm_P0.65mm_EP3.4x6.5mm_Mask2.75x3.43mm_ThermalVias" (at 116.84 26.67 0)
+      (effects (font (size 1.27 1.27)) hide)
+    )
