File: PCB/SmallLedPlatform.kicad_pcb (KiCad board)
At the start: 4 copper layers, 63.5 x 36.1 mm, 121 parts, among them J101 Conn_01x03_Male, J102 USB_C_Receptacle, J103 Conn_01x03_Male, J104 Conn_02x05_Odd_Even, M101 Fan_4pin, Q101 AO3400A, Q201 IRFR7440TRPBF, Q202 IRFR7440TRPBF, Q301 2N7002, Q302 2N7002, Q303 2N7002, Q304 2N7002, SW401 SW_MEC_5E, SW402 SW_MEC_5E, U101 STM32G0B1CBTx, U102 USBLC6-2P6, U103 TCPP01-M12, U201 LM25118, U202 XC6206PxxxMR, U203 WS3222D, U204 WS3222D, U401 AP3722AT

Commit message: Fix review comments
Parts:
- added C108: 100nF/50V, Capacitor_SMD:C_0402_1005Metric, F.Cu at (139.2, 102.9)
- added C109: 1uF/25V, Capacitor_SMD:C_0402_1005Metric, F.Cu at (139.2, 103.9)
- added C403: 100nF/50V, Capacitor_SMD:C_0402_1005Metric, F.Cu at (143.5, 112.3)
- added C404: 100nF/50V, Capacitor_SMD:C_0402_1005Metric, F.Cu at (141.5, 110.2)
- D102: footprint Skrooter_footprints:TVS_ESDA25P35-1U1M -> SkrooterFootprints:TVS_ESDA25P35-1U1M
- D304, D305, D306, D307, D308, D309: footprint Skrooter_footprints:LED_0603_1608Metric_smaller_silk -> SkrooterFootprints:LED_0603_1608Metric_smaller_silk
- U401: footprint Skrooter_footprints:AP3722AT -> SkrooterFootprints:AP3722AT
- moved R403 1.59 mm to (141.5, 111.3), turned to 0 degrees
- moved Q202 0.97 mm to (111.8, 102.5)
- moved Q201 0.90 mm to (106.1, 83.9)
- moved R307 0.89 mm to (140.0, 105.1), turned to 180 degrees
- moved R402 0.85 mm to (141.5, 112.3), turned to 0 degrees
- moved D202 0.85 mm to (110.0, 92.5)
- moved J101 0.76 mm to (144.8, 104.9)
- moved C101 0.63 mm to (142.0, 103.9)
- moved C102 0.42 mm to (141.7, 102.9)
- moved TP201 0.38 mm to (141.2, 107.7)
- moved D301 0.18 mm to (125.4, 87.2)
- moved D311 0.13 mm to (116.2, 92.3)
- moved C201 0.13 mm to (112.8, 85.6)
- moved C222 0.13 mm to (114.8, 85.6)
- moved R101 0.13 mm to (145.2, 102.1)
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- renumbered M101 to M401
Connections:
- net /Power/5V_Sense renamed /5V_Sense
- net /Power/VIN_SENSE renamed /VIN_Sense
- net Net-(U101-Pad45) renamed /Fan_PWM
- net Net-(U101-Pad48) renamed /Fan_Tachomenter
- R213 pad 2: GND -> /HS_EN
- U101 pad 4: unconnected-(U101-Pad4) -> +3V3
- U101 pad 44: unconnected-(U101-Pad44) -> /HS_EN
- U101 pad 5: unconnected-(U101-Pad5) -> /VREF+
Routing:
- net /HS_EN: track 0.00 -> 29.7 mm, vias 0 -> 2
- net GND: track 47.1 -> 51.0 mm, vias 81 -> 84
- net /VREF+: track 0.00 -> 3.08 mm
- net /MCU_SW2: track 32.7 -> 35.8 mm
- net /MCU_SW1: track 37.9 -> 39.8 mm
- net +3V3: track 21.6 -> 22.8 mm
- net /VBUS_CONN: track 25.4 -> 26.4 mm
- net /Power/Power LEDS/15v_gate: track 14.3 -> 15.1 mm
- net /DEBUG_UART_TX: track 4.66 -> 3.89 mm
- net /Power/VIN: track 43.0 -> 43.7 mm
- net SHIELD: vias 98 -> 99

Commit message: Final fixes before production
Connections:
- net /VIN_Sense renamed /VIN_Sense_MCU
Routing:
- net GND: track 51.0 -> 50.7 mm, vias 84 -> 77
Other:
- board text added: "2023-04-02"
- board text removed: "2023-02-11"
