File: PCB/SmallLedPlatform.kicad_sch (KiCad schematic)
At the start: 37 parts, among them J101 Conn_01x03_Male, J102 USB_C_Receptacle, J103 Conn_01x03_Male, J104 Conn_02x05_Odd_Even, Q101 AO3400A, U101 STM32G0B1CBTx, U102 USBLC6-2P6, U103 TCPP01-M12

Commit message: Final fixes before production
Parts:
- D102: symbol Skrooter_symbols:ESDA25P35-1U1M -> Skrooterlib:ESDA25P35-1U1M
- H105, H106, H107: now left out of the parts list
- J101, J103: symbol Connector:Conn_01x03_Male -> Connector:Conn_01x03_Pin
- J102: LCSC C2927300 -> C165948
- R108: LCSC C105871 -> C25867
- U103: symbol Skrooter_symbols:TCPP01-M12 -> Skrooterlib:TCPP01-M12; LCSC (none) -> C1121848
Connections:
- net VIN_Sense renamed VIN_Sense_MCU
Changed lines of the file:
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@@
     (stroke (width 0) (type default))
   )
-  (polyline (pts (xy 207.01 113.03) (xy 207.01 165.1))
+  (polyline (pts (xy 209.55 113.03) (xy 209.55 165.1))
     (stroke (width 0) (type default))
   )
@@
     (effects (font (size 1.27 1.27)) (justify left bottom))
   )
-  (label "VIN_Sense" (at 186.69 62.23 180) (fields_autoplaced)
+  (label "VIN_Sense_MCU" (at 186.69 62.23 180) (fields_autoplaced)
     (effects (font (size 1.27 1.27)) (justify right bottom))
   )
@@
     (effects (font (size 1.27 1.27)) (justify left bottom))
   )
-  (label "VIN_Sense" (at 193.04 135.89 0) (fields_autoplaced)
+  (label "VIN_Sense_MCU" (at 193.04 135.89 0) (fields_autoplaced)
     (effects (font (size 1.27 1.27)) (justify left bottom))
   )
@@
     )
   )
-  (symbol (lib_id "Skrooter_symbols:SHIELD") (at 29.21 96.52 0) (unit 1)
+  (symbol (lib_id "Skrooterlib:SHIELD") (at 29.21 96.52 0) (unit 1)
     (in_bom yes) (on_board yes) (dnp no) (fields_autoplaced)
     (property "Reference" "#PWR0112" (at 29.21 101.6 0)
@@
       (effects (font (size 1.27 1.27)) hide)
     )
-    (property "LCSC" "C2927300" (at 29.21 38.1 0)
+    (property "LCSC" "C165948" (at 29.21 38.1 0)
       (effects (font (size 1.27 1.27)) hide)
     )
@@
     )
   )
-  (symbol (lib_id "Skrooter_symbols:SHIELD") (at 29.21 109.22 0) (unit 1)
+  (symbol (lib_id "Skrooterlib:SHIELD") (at 29.21 109.22 0) (unit 1)
     (in_bom yes) (on_board yes) (dnp no) (fields_autoplaced)
     (property "Reference" "#PWR0115" (at 29.21 114.3 0)
@@
   )
   (symbol (lib_id "Mechanical:MountingHole") (at 17.78 187.96 270) (unit 1)
-    (in_bom yes) (on_board yes) (dnp no)
+    (in_bom no) (on_board yes) (dnp no)
     (property "Reference" "H105" (at 20.32 187.1253 90)
       (effects (font (size 1.27 1.27)) (justify left))
@@
   )
   (symbol (lib_id "Mechanical:MountingHole") (at 55.88 187.96 0) (unit 1)
-    (in_bom yes) (on_board yes) (dnp no) (fields_autoplaced)
+    (in_bom no) (on_board yes) (dnp no) (fields_autoplaced)
     (property "Reference" "H107" (at 58.42 187.1253 0)
       (effects (font (size 1.27 1.27)) (justify left))
@@
     )
   )
-  (symbol (lib_id "Skrooter_symbols:ESDA25P35-1U1M") (at 27.94 149.86 270) (unit 1)
-    (in_bom yes) (on_board yes) (dnp no) (fields_autoplaced)
-    (property "Reference" "D102" (at 29.972 149.0253 90)
-      (effects (font (size 1.27 1.27)) (justify left))
-    )
-    (property "Value" "ESDA25P35-1U1M" (at 29.972 151.5622 90)
+  (symbol (lib_id "Skrooterlib:ESDA25P35-1U1M") (at 27.94 149.86 270) (unit 1)
+    (in_bom yes) (on_board yes) (dnp no) (fields_autoplaced)
+    (property "Reference" "D102" (at 29.972 149.2163 90)
+      (effects (font (size 1.27 1.27)) (justify left))
+    )
+    (property "Value" "ESDA25P35-1U1M" (at 29.972 151.1373 90)
       (effects (font (size 1.27 1.27)) (justify left))
     )
@@
     )
   )
-  (symbol (lib_id "Skrooter_symbols:SHIELD") (at 29.21 120.65 0) (unit 1)
+  (symbol (lib_id "Skrooterlib:SHIELD") (at 29.21 120.65 0) (unit 1)
     (in_bom yes) (on_board yes) (dnp no) (fields_autoplaced)
     (property "Reference" "#PWR0117" (at 29.21 125.73 0)
@@
     )
   )
-  (symbol (lib_id "Connector:Conn_01x03_Male") (at 134.62 29.21 0) (unit 1)
+  (symbol (lib_id "Connector:Conn_01x03_Pin") (at 134.62 29.21 0) (unit 1)
     (in_bom yes) (on_board yes) (dnp no) (fields_autoplaced)
     (property "Reference" "J101" (at 135.255 22.894 0)
@@
     )
   )
-  (symbol (lib_id "Connector:Conn_01x03_Male") (at 153.67 95.25 0) (unit 1)
+  (symbol (lib_id "Connector:Conn_01x03_Pin") (at 153.67 95.25 0) (unit 1)
     (in_bom yes) (on_board yes) (dnp no) (fields_autoplaced)
     (property "Reference" "J103" (at 154.305 88.934 0)
@@
     )
   )
-  (symbol (lib_id "Skrooter_symbols:SHIELD") (at 21.59 68.58 0) (unit 1)
+  (symbol (lib_id "Skrooterlib:SHIELD") (at 21.59 68.58 0) (unit 1)
     (in_bom yes) (on_board yes) (dnp no) (fields_autoplaced)
     (property "Reference" "#PWR0107" (at 21.59 73.66 0)
@@
     )
   )
-  (symbol (lib_id "Skrooter_symbols:SHIELD") (at 55.88 83.82 0) (unit 1)
+  (symbol (lib_id "Skrooterlib:SHIELD") (at 55.88 83.82 0) (unit 1)
     (in_bom yes) (on_board yes) (dnp no) (fields_autoplaced)
     (property "Reference" "#PWR0110" (at 55.88 88.9 0)
@@
     )
   )
-  (symbol (lib_id "Skrooter_symbols:SHIELD") (at 29.21 83.82 0) (unit 1)
+  (symbol (lib_id "Skrooterlib:SHIELD") (at 29.21 83.82 0) (unit 1)
     (in_bom yes) (on_board yes) (dnp no) (fields_autoplaced)
     (property "Reference" "#PWR0109" (at 29.21 88.9 0)
@@
   )
   (symbol (lib_id "Mechanical:MountingHole") (at 38.1 187.96 0) (unit 1)
-    (in_bom yes) (on_board yes) (dnp no) (fields_autoplaced)
+    (in_bom no) (on_board yes) (dnp no) (fields_autoplaced)
     (property "Reference" "H106" (at 40.64 187.1253 0)
       (effects (font (size 1.27 1.27)) (justify left))
@@
     )
   )
-  (symbol (lib_id "Skrooter_symbols:TCPP01-M12") (at 120.65 156.21 0) (unit 1)
+  (symbol (lib_id "Skrooterlib:TCPP01-M12") (at 120.65 156.21 0) (unit 1)
     (in_bom yes) (on_board yes) (dnp no) (fields_autoplaced)
     (property "Reference" "U103" (at 122.6694 152.561 0)
@@
     )
     (property "Datasheet" "" (at 127 154.94 0)
+      (effects (font (size 1.27 1.27)) hide)
+    )
+    (property "LCSC" "C1121848" (at 120.65 156.21 0)
       (effects (font (size 1.27 1.27)) hide)
     )
@@
       (effects (font (size 1.27 1.27)) hide)
     )
-    (property "LCSC" "C105871" (at 165.1 163.83 0)
-      (effects (font (size 1.27 1.27)) hide)
-    )
+    (property "LCSC" "C25867" (at 165.1 163.83 0)
+      (effects (font (size 1.27 1.27)) hide)
+    )
